File: hardware/ps2_to_amiga.kicad_pcb (KiCad board)
At the start: 2 copper layers, 22.9 x 15.2 mm, 6 parts, among them J1 Conn_01x05, J2 Conn_01x04, J3 Conn_02x03_Odd_Even, U1 ATtiny85-20S

Commit message: Add DIN-5 180deg angle footprint
Parts:
- added J4: DIN-5_180degree, Library:DIN_5PIN_180d_Female, F.Cu at (163.8, 81.3)
Changed lines of the file:
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@@
   (net 7 "PS2_DAT")
   (net 8 "/ISP_RST")
+  (net 9 "unconnected-(J4-Pad1)")
+  (net 10 "unconnected-(J4-Pad2)")
+  (net 11 "unconnected-(J4-Pad3)")
+  (net 12 "unconnected-(J4-Pad4)")
+  (net 13 "unconnected-(J4-Pad5)")
+  (footprint "Library:DIN_5PIN_180d_Female" (layer "F.Cu")
+    (at 163.83 81.28)
+    (property "Sheetfile" "ps2_to_amiga.kicad_sch")
+    (property "Sheetname" "")
+    (attr through_hole)
+    (fp_text reference "J4" (at 0 11 unlocked) (layer "F.SilkS")
+      (effects (font (size 1 1) (thickness 0.15)))
+    )
+    (fp_text value "DIN-5_180degree" (at 0 12.5 unlocked) (layer "F.Fab")
+      (effects (font (size 1 1) (thickness 0.15)))
+    )
+    (fp_text user "${REFERENCE}" (at 0 14 unlocked) (layer "F.Fab")
+      (effects (font (size 1 1) (thickness 0.15)))
+    )
+    (fp_line (start -7 -3) (end -7 3) (layer "F.SilkS") (width 0.12))
+    (fp_line (start -7 -9) (end -7 -7) (layer "F.SilkS") (width 0.12))
+    (fp_line (start -7 7) (end -7 9) (layer "F.SilkS") (width 0.12))
+    (fp_rect (start -9.5 9) (end 9.5 -9) (layer "F.SilkS") (width 0.12) (fill none))
+    (pad "1" thru_hole circle (at 3 7.5) (size 2.5 2.5) (drill 1.4) (layers *.Cu *.Mask)
+      (net 9 "unconnected-(J4-Pad1)") (pintype "passive"))
+    (pad "2" thru_hole circle (at 3 0) (size 2.5 2.5) (drill 1.4) (layers *.Cu *.Mask)
+      (net 10 "unconnected-(J4-Pad2)") (pintype "passive"))
+    (pad "3" thru_hole circle (at 3 -7.5) (size 2.5 2.5) (drill 1.4) (layers *.Cu *.Mask)
+      (net 11 "unconnected-(J4-Pad3)") (pintype "passive"))
+    (pad "4" thru_hole circle (at 5.5 5) (size 2.5 2.5) (drill 1.4) (layers *.Cu *.Mask)
+      (net 12 "unconnected-(J4-Pad4)") (pintype "passive"))
+    (pad "5" thru_hole circle (at 5.5 -5) (size 2.5 2.5) (drill 1.4) (layers *.Cu *.Mask)
+      (net 13 "unconnected-(J4-Pad5)") (pintype "passive"))
+    (pad "6" thru_hole circle (at -7 -5) (size 2.5 2.5) (drill 1.4) (layers *.Cu *.Mask))
+    (pad "6" thru_hole circle (at -7 5) (size 2.5 2.5) (drill 1.4) (layers *.Cu *.Mask))
+  )
   (footprint "Connector_PinHeader_2.54mm:PinHeader_2x03_P2.54mm_Vertical" (layer "F.Cu")
     (at 137.16 86.36 90)

Commit message: Design rev2 pcb
Parts:
- removed J3: Conn_02x03_Odd_Even, Connector_PinHeader_2.54mm:PinHeader_2x03_P2.54mm_Vertical
- J1: footprint Connector_PinHeader_2.54mm:PinHeader_1x05_P2.54mm_Vertical -> Library:AMIGA_KB_PADS
- J2: value Conn_01x04 -> AVR-ISP-6; footprint Connector_PinHeader_2.54mm:PinHeader_1x04_P2.54mm_Vertical -> Connector_PinHeader_2.54mm:PinHeader_2x03_P2.54mm_Vertical
- moved J1 8.56 mm to (139.8, 80.0), turned to -90 degrees
- moved U1 8.31 mm to (147.8, 77.8)
- moved REF** 5.47 mm to (148.5, 75.2)
- moved J2 5.31 mm to (150.5, 83.0), turned to -90 degrees
- moved C1 5.17 mm to (147.8, 73.2), turned to 180 degrees
- moved J4 1.53 mm to (163.0, 80.0), turned to 180 degrees
Connections:
- J1 pad 2: AMIGA_RST -> AMIGA_CLK
- J1 pad 4: AMIGA_CLK -> AMIGA_RST
- J2 pad 1: +5V -> PS2_DAT
- J2 pad 2: PS2_CLK -> +5V
- J2 pad 3: PS2_DAT -> PS2_CLK
- J2 pad 4: GND -> AMIGA_RST
- J4 pad 1: unconnected-(J4-Pad1) -> PS2_CLK
- J4 pad 2: unconnected-(J4-Pad2) -> PS2_DAT
- J4 pad 4: unconnected-(J4-Pad4) -> GND
- J4 pad 5: unconnected-(J4-Pad5) -> +5V
- J4 pad 6: (no net) -> GND
- U1 pad 2: AMIGA_RST -> AMIGA_CLK
- U1 pad 5: AMIGA_CLK -> AMIGA_RST
Routing:
- net AMIGA_CLK: track 21.2 -> 3.67 mm, vias 1 -> 0
- net PS2_CLK: track 20.3 -> 34.1 mm, vias 1 -> 0
- net AMIGA_RST: track 4.14 -> 17.0 mm
- net PS2_DAT: track 26.3 -> 14.3 mm, vias 1 -> 0
- net +5V: track 30.4 -> 38.9 mm, vias 1 -> 0
- net /ISP_RST: track 16.8 -> 10.6 mm, vias 1 -> 0
- net AMIGA_DAT: track 4.66 -> 5.77 mm
Other:
- board size 22.9 x 15.2 mm -> 46.8 x 18 mm
- board text added: "rev 2"
- board text removed: "rev 1"
