File: hardware/ps2_to_amiga.kicad_sch (KiCad schematic)
At the start: 5 parts, among them J1 Conn_01x05, J2 Conn_01x04, J3 Conn_02x03_Odd_Even, U1 ATtiny85-20S

Commit message: Add DIN-5 180deg angle footprint
Parts:
- added J4: DIN-5_180degree, Library:DIN_5PIN_180d_Female, symbol Connector:DIN-5_180degree
Changed lines of the file:
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@@
     (pin "6")
+  )
+  (symbol (lib_id "Connector:DIN-5_180degree") (at 161.29 109.22 0) (unit 1)
+    (in_bom yes) (on_board yes) (fields_autoplaced)
+    (property "Reference" "J4" (id 0) (at 161.2901 116.84 0))
+    (property "Value" "DIN-5_180degree" (id 1) (at 161.2901 119.38 0))
+    (property "Footprint" "Library:DIN_5PIN_180d_Female" (id 2) (at 161.29 109.22 0)
+      (effects (font (size 1.27 1.27)) hide)
+    )
+    (property "Datasheet" "http://www.mouser.com/ds/2/18/40_c091_abd_e-75918.pdf" (id 3) (at 161.29 109.22 0)
+      (effects (font (size 1.27 1.27)) hide)
+    )
+    (pin "1")
+    (pin "2")
+    (pin "3")
+    (pin "4")
+    (pin "5")
   )
   (symbol (lib_id "power:+5V") (at 81.28 83.82 0) (mirror y) (unit 1)
@@
       (reference "J3") (unit 1) (value "Conn_02x03_Odd_Even") (footprint "Connector_PinHeader_2.54mm:PinHeader_2x03_P2.54mm_Vertical")
     )
+    (path "/25b9b6d4-722b-4fc2-8315-c355f287841f"
+      (reference "J4") (unit 1) (value "DIN-5_180degree") (footprint "Library:DIN_5PIN_180d_Female")
+    )
     (path "/b75ad8c5-9f55-49ef-9af8-7ab1b11ab9d4"

Commit message: Design rev2 pcb
Parts:
- removed J2: Conn_01x04, Connector_PinHeader_2.54mm:PinHeader_1x04_P2.54mm_Vertical, symbol Connector_Generic:Conn_01x04
- removed J3: Conn_02x03_Odd_Even, Connector_PinHeader_2.54mm:PinHeader_2x03_P2.54mm_Vertical, symbol Connector_Generic:Conn_02x03_Odd_Even
- added J2: AVR-ISP-6, Connector_PinHeader_2.54mm:PinHeader_2x03_P2.54mm_Vertical, symbol Connector:AVR-ISP-6
- J1: footprint Connector_PinHeader_2.54mm:PinHeader_1x05_P2.54mm_Vertical -> Library:AMIGA_KB_PADS
Connections:
- net +5V: now also J4.5, J2.2 (VCC)
- net AMIGA_CLK: now also J1.2 (Pin_2), U1.2 (XTAL1/PB3); no longer J1.4 (Pin_4), U1.5 (AREF/PB0)
- net AMIGA_RST: now also J1.4 (Pin_4), U1.5 (AREF/PB0), J2.4 (MOSI); no longer J1.2 (Pin_2), U1.2 (XTAL1/PB3)
- net GND: now also J4.4, J4.6, J2.6 (GND)
- net ISP_RST: now also J2.5 (~{RST})
- net PS2_CLK: now also J4.1, J2.3 (SCK)
- net PS2_DAT: now also J4.2, J2.1 (MISO)
- no-connect marks 0 -> 2
